Commit message: Added lidar sensor, contact sensor, and gazebo launcher file

File: robot/control.xacro (robot description, xacro)
@@ -1,6 +1,42 @@
 <?xml version="1.0"?>
 <robot xmlns:xacro="http://www.ros.org/wiki/xacro" >
-<!-- =================================================================================== -->
-<!-- |    This XACRO contains physical elements (the chassis and wheels ) of the robot | -->
-<!-- =================================================================================== -->
+    <!-- =================================================================================== -->
+    <!-- |    This XACRO contains physical elements (the chassis and wheels ) of the robot | -->
+    <!-- =================================================================================== -->
+    <gazebo>
+        <plugin name="diff_drive" filename="libgazebo_ros_diff_drive.so">
+            <!-- Plugin update rate in Hz -->
+            <updateRate>30.0</updateRate>
+            <!-- Name of left joint, defaults to `left_joint` -->
+            <leftJoint>left_wheel_joint</leftJoint>
+            <!-- Name of right joint, defaults to `right_joint` -->
+            <rightJoint>right_wheel_joint</rightJoint>
+            <!-- The distance from the center of one wheel to the other, in meters, defaults to 0.34 m -->
+            <wheelSeparation>0.350</wheelSeparation>
+            <!-- Diameter of the wheels, in meters, defaults to 0.15 m -->
+            <wheelDiameter>0.10</wheelDiameter>
+            <!-- Wheel acceleration, in rad/s^2, defaults to 0.0 rad/s^2 -->
+            <wheelAcceleration>1.0</wheelAcceleration>
+            <!-- Maximum torque which the wheels can produce, in Nm, defaults to 5 Nm -->
+            <wheelTorque>20</wheelTorque>
+            <!-- Topic to receive geometry_msgs/Twist message commands, defaults to `cmd_vel` -->
+            <commandTopic>cmd_vel</commandTopic>
+            <!-- Topic to publish nav_msgs/Odometry messages, defaults to `odom` -->
+            <odometryTopic>odom</odometryTopic>
+            <!-- Odometry frame, defaults to `odom` -->
+            <odometryFrame>odom</odometryFrame>
+            <!-- Robot frame to calculate odometry from, defaults to `base_footprint` -->
+            <robotBaseFrame>base_footprint</robotBaseFrame>
+            <!-- Odometry source, 0 for ENCODER, 1 for WORLD, defaults to WORLD -->
+            <odometrySource>1</odometrySource>
+            <!-- Set to true to publish transforms for the wheel links, defaults to false -->
+            <publishWheelTF>true</publishWheelTF>
+            <!-- Set to true to publish transforms for the odometry, defaults to true -->
+            <publishOdom>true</publishOdom>
+            <!-- Set to true to publish sensor_msgs/JointState on /joint_states for the wheel joints, defaults to false -->
+            <publishWheelJointState>true</publishWheelJointState>
+            <!-- Set to true to swap right and left wheels, defaults to true -->
+            <legacyMode>false</legacyMode>
+        </plugin>
+    </gazebo>
 </robot>

File: robot/materials.xacro (robot description, xacro)
@@ -7,5 +7,11 @@
         <material name="blue">
             <!-- The colors are RGB plus alpha (transparency) -->
-            <color rgba="0 0 1 0.5" />
+            <color rgba="0 0 1 1.0" />
+        </material>
+    </xacro:macro>
+    <xacro:macro name="white_material">
+        <material name="white">
+            <!-- The colors are RGB plus alpha (transparency) -->
+            <color rgba="0 0 1 1.0" />
         </material>
     </xacro:macro>
@@ -16,3 +22,19 @@
         </material>
     </xacro:macro>
+    <!-- Gazebo Materials -->
+    <xacro:macro name="blue_gazebo_material" params="object">
+        <gazebo reference="${object}">
+            <material>Gazebo/Blue</material>
+        </gazebo>
+    </xacro:macro>
+    <xacro:macro name="white_gazebo_material" params="object">
+        <gazebo reference="${object}">
+            <material>Gazebo/White</material>
+        </gazebo>
+    </xacro:macro>
+    <xacro:macro name="black_gazebo_material" params="object">
+        <gazebo reference="${object}">
+            <material>Gazebo/Blue</material>
+        </gazebo>
+    </xacro:macro>
 </robot>

File: robot/robot.urdf (robot description, URDF)
Before this commit: robot robot, 5 links, 4 joints
Links:
- added link hokuyo_link, mass 0.1; collision cylinder length=0.04 radius=0.05; visual cylinder length=0.04 radius=0.05
Joints:
- added joint laser_joint: type fixed, parent chassis, child hokuyo_link, origin xyz=0.1 0 0.175 rpy=0 0 0

File: robot/robot.xacro (robot description, xacro)
@@ -5,3 +5,4 @@
     <!-- =================================================================================== -->
     <xacro:include filename="/home/enrique/catkin_ws/src/algorithm/models/robot/robot_core.xacro" />
+    <xacro:include filename="/home/enrique/catkin_ws/src/algorithm/models/robot/control.xacro" />
 </robot>

File: robot/robot_core.xacro (robot description, xacro)
@@ -6,4 +6,5 @@
     <xacro:include filename="/home/enrique/catkin_ws/src/algorithm/models/robot/materials.xacro" />
     <xacro:include filename="/home/enrique/catkin_ws/src/algorithm/models/robot/inertial_macros.xacro" />
+    <xacro:include filename="/home/enrique/catkin_ws/src/algorithm/models/robot/sensors.xacro" />
     <!--BASE LINK-->
     <link name="base_link">
@@ -27,5 +28,5 @@
             <xacro:blue_material />
         </visual>
-        <collision>
+        <collision name="chassis_link_bump_sensor_collision">
             <!-- Origin of the box -->
             <origin xyz="0.15 0 0.075" />
@@ -39,4 +40,5 @@
         </xacro:inertial_box>
     </link>
+    <xacro:blue_gazebo_material object="chassis" />
     <!-- LEFT WHEEL JOINT-->
     <joint name="left_wheel_joint" type="continuous">
@@ -53,5 +55,5 @@
             <xacro:blue_material />
         </visual>
-        <collision>
+        <collision name="left_wheel_link_bump_sensor_collision">
             <geometry>
                 <cylinder radius="0.05" length="0.04" />
@@ -62,4 +64,5 @@
         </xacro:inertial_cylinder>
     </link>
+    <xacro:blue_gazebo_material object="left_wheel" />
     <!-- RIGHT WHEEL JOINT-->
     <joint name="right_wheel_joint" type="continuous">
@@ -76,5 +79,5 @@
             <xacro:blue_material />
         </visual>
-        <collision>
+        <collision name="right_wheel_link_bump_sensor_collision">
             <geometry>
                 <cylinder radius="0.05" length="0.04" />
@@ -85,4 +88,5 @@
         </xacro:inertial_cylinder>
     </link>
+    <xacro:blue_gazebo_material object="right_wheel" />
     <!-- CASTER WHEEL LINK -->
     <joint name="caster_wheel_joint" type="fixed">
@@ -107,3 +111,9 @@
         </xacro:inertial_sphere>
     </link>
+    <xacro:black_gazebo_material object="caster_wheel" />
+    <gazebo reference="caster_wheel">
+        <!-- Reduce the friction of the caster wheel with the enviroment -->
+        <mu1 value="0.001" />
+        <mu2 value="0.001" />
+    </gazebo>
 </robot>
